Commit message: 05292302

File: sim/model/indy7.urdf (robot description, URDF)
Before this commit: robot indy7, 9 links, 8 joints
Links:
- link tcp: mass 0 -> 0.0001

Commit message: 20230618_231443

File: sim/model/indy7.urdf (robot description, URDF)
Before this commit: robot indy7, 9 links, 8 joints
Links:
- link tcp: mass 0.0001 -> 0.0000
